File: Hardware/lx-deciim/switches.kicad_sch (KiCad schematic)
At the start: 12 parts

Commit message: fix: fix mouser part number on schematic + fill page settings
Other:
- company: (none) -> Lucas Bonvin
- title: (none) -> lx-deciim
Changed lines of the file:
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@@
 	(generator_version "9.0")
 	(paper "A4")
+	(title_block
+		(title "lx-deciim")
+		(date "2025-06-17")
+		(rev "v1.0.0")
+		(company "Lucas Bonvin")
+		(comment 1 "This project is licensed under the CC BY-NC 4.0 License.")
+	)
 	(wire
 		(pts
